File: hardware/PicoROM.kicad_sch (KiCad schematic)
At the start: 56 parts, among them J1 USB_C_Receptacle_USB2.0, J2 External Reset, J3 Conn_01x16, J4 Conn_01x16, J5 Conn_01x05_Pin, U1 AP2112K-3.3, U10 74LVCH8T245, U2 W25Q16JVUXIQ, U3 RP2040, U4 74LVCH245, U5 74LVCH245, U7 TCA5405RUGR, U8 74AHCT1G126, U9 74LVCH245, Y1 445C25D12M00000

Commit message: Redesigned ROM emulator.
Changes from the original:
- 4 layer PCB (not 6)
- different level shifters
- 0402 resistors and caps
- reworked ~OE for level shifters
- added fiducials
- different pin solution

TODO:
- make sure USB is impedance matched
- review board outline, tweak if necessary
Parts:
- removed C1, C4: 1u, Capacitor_SMD:C_0805_2012Metric, symbol Device:C
- removed C10, C25, C8: 1u, Capacitor_SMD:C_0402_1005Metric, symbol Device:C
- removed C11, C12, C13, C14, C15, C16, C17, C18, C19, C20, C21, C22, C23, C24, C5, C6, C7, C9: 100n, Capacitor_SMD:C_0201_0603Metric, symbol Device:C
- removed C2, C3: 27p, Capacitor_SMD:C_0402_1005Metric, symbol Device:C
- removed J3, J4: Conn_01x16, Connector_PinHeader_2.54mm:PinHeader_1x16_P2.54mm_Vertical, symbol Connector_Generic:Conn_01x16
- removed R1, R10, R2, R5, R8, R9: 1k, Resistor_SMD:R_0201_0603Metric, symbol Device:R
- removed R11: 100k, Resistor_SMD:R_0201_0603Metric, symbol Device:R
- removed R3, R4: 27, Resistor_SMD:R_0201_0603Metric, symbol Device:R
- removed R6, R7: 5.1k, Resistor_SMD:R_0201_0603Metric, symbol Device:R
- removed U10: 74LVCH8T245, RP2040_minimal:DHVQFN24_L5.5-W3.5-P0.50-BL-EP, symbol Logic_LevelTranslator:SN74AVC8T245PW
- removed U4, U5, U9: 74LVCH245, RP2040_minimal:V-QFN4525-20_L4.5-W2.5-P0.50-BL, symbol 74xx:74LS245
- added C1, C10, C11, C12, C13, C16, C17, C18, C19, C20, C23, C24, C4, C5, C6, C7, C8, C9: 1u, Capacitor_SMD:C_0402_1005Metric_Pad0.74x0.62mm_HandSolder, symbol Device:C_Small
- added C2, C3: 27p, Capacitor_SMD:C_0402_1005Metric_Pad0.74x0.62mm_HandSolder, symbol Device:C_Small
- added FID1, FID10, FID11, FID12, FID2, FID3, FID4, FID5, FID6, FID7, FID8, FID9: Fiducial, UNIC:Fiducial_0.5mm_Mask1mm, symbol Mechanical:Fiducial
- added J6: Conn_02x16_Counter_Clockwise, UNIC:DIP-32_pin_header, symbol Connector_Generic:Conn_02x16_Counter_Clockwise
- added Q1: 2N7002, Package_TO_SOT_SMD:SOT-23, symbol Transistor_FET:2N7002
- added R1, R10, R11, R2, R4, R9: 1k, Resistor_SMD:R_0402_1005Metric_Pad0.72x0.64mm_HandSolder, symbol Device:R_Small_US
- added R12, R6: 5.1k, Resistor_SMD:R_0402_1005Metric_Pad0.72x0.64mm_HandSolder, symbol Device:R_Small_US
- added R3, R5: 27, Resistor_SMD:R_0402_1005Metric_Pad0.72x0.64mm_HandSolder, symbol Device:R_Small_US
- added R7: 100k, Resistor_SMD:R_0402_1005Metric_Pad0.72x0.64mm_HandSolder, symbol Device:R_Small_US
- added R8: 10k, Resistor_SMD:R_0402_1005Metric_Pad0.72x0.64mm_HandSolder, symbol Device:R_Small_US
- added U4, U5, U6: 74CBTD3861, Package_SO:TSSOP-24_4.4x5mm_P0.4mm, symbol 74xx:74CBTD3861
- J2: footprint Connector_PinHeader_2.54mm:PinHeader_1x01_P2.54mm_Vertical -> TestPoint:TestPoint_Pad_D3.0mm
Connections:
- net +1V1: now also C6.1, C7.1, C8.1
- net +3V3: now also C1.1, C10.1, C11.1, C12.1, C13.1, C16.1, C18.1, C24.1, C4.1, C9.1, Q1.1 (G), R4.2, R7.2
- net +5V: now also C17.1, C19.1, C20.1, C23.1, C5.1, R8.2, U4.24 (VCC), U5.24 (VCC), U6.24 (VCC)
- net A0: now also U5.6 (A5)
- net A1: now also U6.22 (B1)
- net A10: now also U6.15 (B8)
- net A11: now also U6.13 (B10)
- net A12: now also U4.11 (A10)
- net A13: now also U4.4 (A3)
- net A14: now also U4.5 (A4)
- net A15: now also U4.10 (A9)
- net A16: now also U4.9 (A8)
- net A17: now also U4.6 (A5)
- net A2: now also U6.21 (B2)
- net A3: now also U6.20 (B3)
- net A4: now also U6.19 (B4)
- net A5: now also U6.18 (B5)
- net A6: now also U6.17 (B6)
- net A7: now also U6.16 (B7)
- net A8: now also U4.3 (A2)
- net A9: now also U4.2 (A1)
- net D0: now also U5.4 (A3)
- net D1: now also U5.3 (A2)
- net D2: now also U5.2 (A1)
- net D3: now also U5.5 (A4)
- net D4: now also U5.7 (A6)
- net D5: now also U5.8 (A7)
- net D6: now also U5.9 (A8)
- net D7: now also U5.10 (A9)
- net EXT_RESET: now also R10.2
- net GND: now also C1.2, C10.2, C11.2, C12.2, C13.2, C16.2, C17.2, C18.2, C19.2, C2.1, C20.2, C23.2, C24.2, C3.1, C4.2, C5.2, C6.2, C7.2, C8.2, C9.2, J6.16 (Pin_16), Q1.2 (S), R12.2, R6.2, U4.12 (GND), U5.12 (GND), U6.12 (GND)
- net INFO_LED1: now also R2.2
- net INFO_LED2: now also R9.2
- net PIN_5V: now also J6.32 (Pin_32)
- net PIN_A0: now also J6.12 (Pin_12), U5.19 (B4)
- net PIN_A1: now also J6.11 (Pin_11), U6.2 (A1)
- net PIN_A10: now also J6.23 (Pin_23), U6.9 (A8)
- net PIN_A11: now also J6.25 (Pin_25), U6.11 (A10)
- net PIN_A12: now also J6.4 (Pin_4), U4.13 (B10)
- net PIN_A13: now also J6.28 (Pin_28), U4.20 (B3)
- net PIN_A14: now also J6.29 (Pin_29), U4.19 (B4)
- net PIN_A15: now also J6.3 (Pin_3), U4.14 (B9)
- net PIN_A16: now also J6.2 (Pin_2), U4.15 (B8)
- net PIN_A17: now also J6.30 (Pin_30), U4.18 (B5)
- net PIN_A2: now also J6.10 (Pin_10), U6.3 (A2)
- net PIN_A3: now also J6.9 (Pin_9), U6.4 (A3)
- net PIN_A4: now also J6.8 (Pin_8), U6.5 (A4)
- net PIN_A5: now also J6.7 (Pin_7), U6.6 (A5)
- net PIN_A6: now also J6.6 (Pin_6), U6.7 (A6)
- net PIN_A7: now also J6.5 (Pin_5), U6.8 (A7)
- net PIN_A8: now also J6.27 (Pin_27), U4.21 (B2)
- net PIN_A9: now also J6.26 (Pin_26), U4.22 (B1)
- net PIN_D0: now also J6.13 (Pin_13), U5.20 (B3)
- net PIN_D1: now also J6.14 (Pin_14), U5.21 (B2)
- net PIN_D2: now also J6.15 (Pin_15), U5.22 (B1)
- net PIN_D3: now also J6.17 (Pin_17), U5.18 (B5)
- net PIN_D4: now also J6.18 (Pin_18), U5.17 (B6)
- net PIN_D5: now also J6.19 (Pin_19), U5.16 (B7)
- net PIN_D6: now also J6.20 (Pin_20), U5.15 (B8)
- net PIN_D7: now also J6.21 (Pin_21), U5.14 (B9)
- net QSPI_SS: now also R11.2
- net USB_D+: now also R5.2
- net USB_D-: now also R3.2
- net XIN: now also C3.2
- net XOUT: now also R1.2
- net ~{CE}: now also R7.1, U5.11 (A10)
- net ~{OE}: now also U6.14 (B9)
- net ~{PIN_CE}: now also J6.22 (Pin_22), U5.13 (B10)
- net ~{PIN_OE}: now also J6.24 (Pin_24), U6.10 (A9)
- net ~{USB_BOOT}: now also R11.1
- net at U3.46 (USB_DM): now also R3.1
- net at U3.47 (USB_DP): now also R5.1
- net at Y1.2: now also C2.2, R1.1
- net at D3.2 (A): now also R9.1
- net at U8.4: now also R10.1
- net at D2.2 (A): now also R2.1
- net at D1.2 (A): now also R4.1
- net at J1.A5 (CC1): now also R6.1
- net at J1.B5 (CC2): now also R12.1
- net ~{BUF_OE}: no longer names the net of U3.30 (GPIO19)
- new net ~{BUF_EN}: Q1.3 (D), R8.1, U4.23 (~{OE}), U5.23 (~{OE}), U6.23 (~{OE})
- no-connect marks 14 -> 6
Other:
- note removed: "Make sure C10 is close to pin 44 of RP2040"
- note removed: "Make sure C8 is close to pin 45 of RP2040"
